File: shield/mod-arduino-shield.sch (KiCad schematic (older format))
At the start: 48 parts, among them J1 RJHSE-5084, J2 RJHSE-5084, Q1 MMBT3904, U1 SN75176BDR

Commit message: removing local copy of footprints and adding the mod-kicad-footprints repository as a submodule dependency
Parts:
- AD1, AD_PROTO1: footprint mod-arduino-shield-lib:HEADER_100MIL_1R6P_PTH -> MOD_Footprints_Lib:HEADER_100MIL_1R6P_PTH
- C1, C7, C9: footprint mod-arduino-shield-lib:CAP_RAD_5MM -> MOD_Footprints_Lib:CAP_RAD_5MM
- C2, C3, C4, C5, C6, C8, R1, R10, R11, R12, R13, R14, R15, R16, R2, R3, R4, R5, R6, R7, R8, R9: footprint mod-arduino-shield-lib:SM0805 -> MOD_Footprints_Lib:SM0805
- D1: footprint mod-arduino-shield-lib:DO-214AC(SMA) -> MOD_Footprints_Lib:DO-214AC(SMA)
- D2, D3: footprint mod-arduino-shield-lib:SOD123 -> MOD_Footprints_Lib:SOD123
- H1: footprint mod-arduino-shield-lib:HOLE_3MM -> MOD_Footprints_Lib:HOLE_3MM
- IOH1, IOH_PROTO1: footprint mod-arduino-shield-lib:HEADER_100MIL_1R10P_PTH -> MOD_Footprints_Lib:HEADER_100MIL_1R10P_PTH
- IOL1, IOL_PROTO1, POWER1, POWER_PROTO1: footprint mod-arduino-shield-lib:HEADER_100MIL_1R8P_PTH -> MOD_Footprints_Lib:HEADER_100MIL_1R8P_PTH
- J1, J2: footprint mod-arduino-shield-lib:RJ45-RJHSE5084 -> MOD_Footprints_Lib:RJ45-RJHSE5084
- JP1: footprint mod-arduino-shield-lib:HEADER_100MIL_2R3P_PTH -> MOD_Footprints_Lib:HEADER_100MIL_2R3P_PTH
- JP2: footprint mod-arduino-shield-lib:HEADER_100MIL_1R2P_PTH -> MOD_Footprints_Lib:HEADER_100MIL_1R2P_PTH
- PROTOBOARD1: footprint mod-arduino-shield-lib:PROTOBOARD_100MIL_8R16P_PTH -> MOD_Footprints_Lib:PROTOBOARD_100MIL_8R16P_PTH
- PROTO_3.3V1, PROTO_5V1, PROTO_GND1: footprint mod-arduino-shield-lib:PROTOBOARD_100MIL_1R16P_PTH -> MOD_Footprints_Lib:PROTOBOARD_100MIL_1R16P_PTH
- Q1: footprint mod-arduino-shield-lib:SOT23 -> MOD_Footprints_Lib:SOT23
- RT1: footprint mod-arduino-shield-lib:SM1210 -> MOD_Footprints_Lib:SM1210
- U1: footprint mod-arduino-shield-lib:SO8E -> MOD_Footprints_Lib:SO8E
