File: hw-design/board/control-chain.sch (KiCad schematic (older format))
At the start: 19 parts, among them J1 CC_INPUT, J2 CC_OUTPUT, Q2 2N7002, Q3 2N7002, Q4 IRFML8244TRPBF, U1 ISL83491

Commit message: adding footprint to local project directory (submodule)
Parts:
- R11: value R -> 10K; footprint (none) -> Resistors_SMD:R_0603; MPN (none) -> RMCF0603JT10K0
Changed lines of the file:
@@
 $EndComp
 $Comp
-L GNDD #PWR018
+L GNDD #PWR020
 U 1 1 557962A0
 P 3750 2500
-F 0 "#PWR018" H 3750 2250 60  0001 C CNN
+F 0 "#PWR020" H 3750 2250 60  0001 C CNN
 F 1 "GNDD" H 3750 2350 60  0000 C CNN
 F 2 "" H 3750 2500 60  0000 C CNN
@@
 $EndComp
 $Comp
-L GNDD #PWR019
+L GNDD #PWR021
 U 1 1 55797530
 P 3750 4300
-F 0 "#PWR019" H 3750 4050 60  0001 C CNN
+F 0 "#PWR021" H 3750 4050 60  0001 C CNN
 F 1 "GNDD" H 3750 4150 60  0000 C CNN
 F 2 "" H 3750 4300 60  0000 C CNN
@@
 $EndComp
 $Comp
-L GNDD #PWR020
+L GNDD #PWR022
 U 1 1 557A784F
 P 4950 4650
-F 0 "#PWR020" H 4950 4400 60  0001 C CNN
+F 0 "#PWR022" H 4950 4400 60  0001 C CNN
 F 1 "GNDD" H 4950 4500 60  0000 C CNN
 F 2 "" H 4950 4650 60  0000 C CNN
@@
 $EndComp
 $Comp
-L +9V #PWR021
+L +9V #PWR023
 U 1 1 557AE435
 P 4950 3550
-F 0 "#PWR021" H 4950 3400 50  0001 C CNN
+F 0 "#PWR023" H 4950 3400 50  0001 C CNN
 F 1 "+9V" H 4950 3690 50  0000 C CNN
 F 2 "" H 4950 3550 60  0000 C CNN
@@
 $EndComp
 $Comp
-L +9V #PWR022
+L +9V #PWR024
 U 1 1 557B6A6D
 P 4400 3550
-F 0 "#PWR022" H 4400 3400 50  0001 C CNN
+F 0 "#PWR024" H 4400 3400 50  0001 C CNN
 F 1 "+9V" H 4400 3690 50  0000 C CNN
 F 2 "" H 4400 3550 60  0000 C CNN
@@
 $EndComp
 $Comp
-L +9V #PWR023
+L +9V #PWR025
 U 1 1 557B80CC
 P 4400 1750
-F 0 "#PWR023" H 4400 1600 50  0001 C CNN
+F 0 "#PWR025" H 4400 1600 50  0001 C CNN
 F 1 "+9V" H 4400 1890 50  0000 C CNN
 F 2 "" H 4400 1750 60  0000 C CNN
@@
 $EndComp
 $Comp
-L GNDD #PWR024
+L GNDD #PWR026
 U 1 1 557D6D91
 P 7850 3200
-F 0 "#PWR024" H 7850 2950 60  0001 C CNN
+F 0 "#PWR026" H 7850 2950 60  0001 C CNN
 F 1 "GNDD" H 7850 3050 60  0000 C CNN
 F 2 "" H 7850 3200 60  0000 C CNN
@@
 $EndComp
 $Comp
-L +3.3V #PWR025
+L +3.3V #PWR027
 U 1 1 557D9E83
 P 8150 1600
-F 0 "#PWR025" H 8150 1450 50  0001 C CNN
+F 0 "#PWR027" H 8150 1450 50  0001 C CNN
 F 1 "+3.3V" H 8150 1740 50  0000 C CNN
 F 2 "" H 8150 1600 60  0000 C CNN
@@
 $EndComp
 $Comp
-L GNDD #PWR026
+L GNDD #PWR028
 U 1 1 557DFB58
 P 8650 3300
-F 0 "#PWR026" H 8650 3050 60  0001 C CNN
+F 0 "#PWR028" H 8650 3050 60  0001 C CNN
 F 1 "GNDD" H 8650 3150 60  0000 C CNN
 F 2 "" H 8650 3300 60  0000 C CNN
@@
 $EndComp
 $Comp
-L GNDD #PWR027
+L GNDD #PWR029
 U 1 1 557A1AB4
 P 2450 6900
-F 0 "#PWR027" H 2450 6650 60  0001 C CNN
+F 0 "#PWR029" H 2450 6650 60  0001 C CNN
 F 1 "GNDD" H 2450 6750 60  0000 C CNN
 F 2 "" H 2450 6900 60  0000 C CNN
@@
 $EndComp
 $Comp
-L +9V #PWR028
+L +9V #PWR030
 U 1 1 557A4EDD
 P 2450 5800
-F 0 "#PWR028" H 2450 5650 50  0001 C CNN
+F 0 "#PWR030" H 2450 5650 50  0001 C CNN
 F 1 "+9V" H 2450 5940 50  0000 C CNN
 F 2 "" H 2450 5800 60  0000 C CNN
@@
 $EndComp
 $Comp
-L GNDD #PWR029
+L GNDD #PWR031
 U 1 1 557B0B8B
 P 4300 6900
-F 0 "#PWR029" H 4300 6650 60  0001 C CNN
+F 0 "#PWR031" H 4300 6650 60  0001 C CNN
 F 1 "GNDD" H 4300 6750 60  0000 C CNN
 F 2 "" H 4300 6900 60  0000 C CNN
@@
 $EndComp
 $Comp
-L +9V #PWR030
+L +9V #PWR032
 U 1 1 557B0B9A
 P 4300 5800
-F 0 "#PWR030" H 4300 5650 50  0001 C CNN
+F 0 "#PWR032" H 4300 5650 50  0001 C CNN
 F 1 "+9V" H 4300 5940 50  0000 C CNN
 F 2 "" H 4300 5800 60  0000 C CNN
@@
 $EndComp
 $Comp
-L +9V #PWR031
+L +9V #PWR033
 U 1 1 557B22CB
 P 2150 3300
-F 0 "#PWR031" H 2150 3150 50  0001 C CNN
+F 0 "#PWR033" H 2150 3150 50  0001 C CNN
 F 1 "+9V" H 2150 3440 50  0000 C CNN
 F 2 "" H 2150 3300 60  0000 C CNN
@@
 $EndComp
 $Comp
-L +9V #PWR032
+L +9V #PWR034
 U 1 1 557B2849
 P 2150 4000
-F 0 "#PWR032" H 2150 3850 50  0001 C CNN
+F 0 "#PWR034" H 2150 3850 50  0001 C CNN
 F 1 "+9V" H 2150 4140 50  0000 C CNN
 F 2 "" H 2150 4000 60  0000 C CNN
@@
 $EndComp
 $Comp
-L +9V #PWR033
+L +9V #PWR035
 U 1 1 557B3090
 P 2150 2200
-F 0 "#PWR033" H 2150 2050 50  0001 C CNN
+F 0 "#PWR035" H 2150 2050 50  0001 C CNN
 F 1 "+9V" H 2150 2340 50  0000 C CNN
 F 2 "" H 2150 2200 60  0000 C CNN
@@
 $EndComp
 $Comp
-L +9V #PWR034
+L +9V #PWR036
 U 1 1 557B39CA
 P 2150 1500
-F 0 "#PWR034" H 2150 1350 50  0001 C CNN
+F 0 "#PWR036" H 2150 1350 50  0001 C CNN
 F 1 "+9V" H 2150 1640 50  0000 C CNN
 F 2 "" H 2150 1500 60  0000 C CNN
@@
 $EndComp
 $Comp
-L GNDD #PWR035
+L GNDD #PWR037
 U 1 1 557F118D
 P 8650 2350
-F 0 "#PWR035" H 8650 2100 60  0001 C CNN
+F 0 "#PWR037" H 8650 2100 60  0001 C CNN
 F 1 "GNDD" H 8650 2200 60  0000 C CNN
 F 2 "" H 8650 2350 60  0000 C CNN
@@
 P 9250 1850
 F 0 "R11" V 9330 1850 50  0000 C CNN
-F 1 "R" V 9250 1850 50  0000 C CNN
-F 2 "" V 9180 1850 30  0000 C CNN
+F 1 "10K" V 9250 1850 50  0000 C CNN
+F 2 "Resistors_SMD:R_0603" V 9180 1850 30  0000 C CNN
 F 3 "" H 9250 1850 30  0000 C CNN
+F 4 "RMCF0603JT10K0" V 9250 1850 60  0001 C CNN "MPN"
 	1    9250 1850
 	1    0    0    -1
@@
 Connection ~ 9250 2100
 $Comp
-L +3.3V #PWR036
+L +3.3V #PWR038
 U 1 1 558CADB4
 P 9250 1600
-F 0 "#PWR036" H 9250 1450 50  0001 C CNN
+F 0 "#PWR038" H 9250 1450 50  0001 C CNN
 F 1 "+3.3V" H 9250 1740 50  0000 C CNN
 F 2 "" H 9250 1600 60  0000 C CNN

Commit message: sch: changing input voltage from +9V to +12V
Parts:
- removed R6, R7: 10k, Resistors_SMD:R_0603, symbol R
- R2, R3, R4, R5: value 820R -> 1K; MPN ESR03EZPJ821 -> ESR03EZPJ102
Connections:
- net +9V renamed +12V
Other:
- moved on the sheet: Q2, Q3
Changed lines of the file:
@@
-$EndComp
-$Comp
-L +9V #PWR023
-U 1 1 557AE435
-P 4950 3550
-F 0 "#PWR023" H 4950 3400 50  0001 C CNN
-F 1 "+9V" H 4950 3690 50  0000 C CNN
-F 2 "" H 4950 3550 60  0000 C CNN
-F 3 "" H 4950 3550 60  0000 C CNN
-	1    4950 3550
-	1    0    0    -1
-$EndComp
-$Comp
-L +9V #PWR024
-U 1 1 557B6A6D
-P 4400 3550
-F 0 "#PWR024" H 4400 3400 50  0001 C CNN
-F 1 "+9V" H 4400 3690 50  0000 C CNN
-F 2 "" H 4400 3550 60  0000 C CNN
-F 3 "" H 4400 3550 60  0000 C CNN
-	1    4400 3550
-	1    0    0    -1
-$EndComp
-$Comp
-L +9V #PWR025
-U 1 1 557B80CC
-P 4400 1750
-F 0 "#PWR025" H 4400 1600 50  0001 C CNN
-F 1 "+9V" H 4400 1890 50  0000 C CNN
-F 2 "" H 4400 1750 60  0000 C CNN
-F 3 "" H 4400 1750 60  0000 C CNN
-	1    4400 1750
-	1    0    0    -1
 $EndComp
 $Comp
@@
 P 2400 3400
 F 0 "R4" V 2480 3400 50  0000 C CNN
-F 1 "820R" V 2400 3400 50  0000 C CNN
+F 1 "1K" V 2400 3400 50  0000 C CNN
 F 2 "Resistors_SMD:R_0603" V 2330 3400 30  0000 C CNN
 F 3 "" H 2400 3400 30  0000 C CNN
-F 4 "ESR03EZPJ821" H 0   0   50  0001 C CNN "MPN"
+F 4 "ESR03EZPJ102" H 0   0   50  0001 C CNN "MPN"
 	1    2400 3400
 	0    1    -1   0
@@
 P 2400 1600
 F 0 "R2" V 2480 1600 50  0000 C CNN
-F 1 "820R" V 2400 1600 50  0000 C CNN
+F 1 "1K" V 2400 1600 50  0000 C CNN
 F 2 "Resistors_SMD:R_0603" V 2330 1600 30  0000 C CNN
 F 3 "" H 2400 1600 30  0000 C CNN
-F 4 "ESR03EZPJ821" H 0   0   50  0001 C CNN "MPN"
+F 4 "ESR03EZPJ102" H 0   0   50  0001 C CNN "MPN"
 	1    2400 1600
 	0    1    -1   0
@@
 P 2400 4100
 F 0 "R5" V 2480 4100 50  0000 C CNN
-F 1 "820R" V 2400 4100 50  0000 C CNN
+F 1 "1K" V 2400 4100 50  0000 C CNN
 F 2 "Resistors_SMD:R_0603" V 2330 4100 30  0000 C CNN
 F 3 "" H 2400 4100 30  0000 C CNN
-F 4 "ESR03EZPJ821" H 0   0   50  0001 C CNN "MPN"
+F 4 "ESR03EZPJ102" H 0   0   50  0001 C CNN "MPN"
 	1    2400 4100
 	0    1    -1   0
@@
 P 2400 2300
 F 0 "R3" V 2480 2300 50  0000 C CNN
-F 1 "820R" V 2400 2300 50  0000 C CNN
+F 1 "1K" V 2400 2300 50  0000 C CNN
 F 2 "Resistors_SMD:R_0603" V 2330 2300 30  0000 C CNN
 F 3 "" H 2400 2300 30  0000 C CNN
-F 4 "ESR03EZPJ821" H 0   0   50  0001 C CNN "MPN"
+F 4 "ESR03EZPJ102" H 0   0   50  0001 C CNN "MPN"
 	1    2400 2300
 	0    1    -1   0
@@
 L Q_NMOS_GSD Q2
 U 1 1 557A16B1
-P 2350 6600
-F 0 "Q2" H 2250 6650 50  0000 R CNN
-F 1 "2N7002" V 2550 6750 50  0000 R CNN
-F 2 "Housings_SOT-23_SOT-143_TSOT-6:SOT-23" H 2550 6700 29  0000 C CNN
-F 3 "" H 2350 6600 60  0000 C CNN
-F 4 "2N7002P,215" H 0   0   50  0001 C CNN "MPN"
-	1    2350 6600
+P 2200 6100
+F 0 "Q2" H 2100 6150 50  0000 R CNN
+F 1 "2N7002" V 2400 6250 50  0000 R CNN
+F 2 "Housings_SOT-23_SOT-143_TSOT-6:SOT-23" H 2400 6200 29  0000 C CNN
+F 3 "" H 2200 6100 60  0000 C CNN
+F 4 "2N7002P,215" H -150 -500 50  0001 C CNN "MPN"
+	1    2200 6100
 	1    0    0    -1
 $EndComp
@@
 L GNDD #PWR029
 U 1 1 557A1AB4
-P 2450 6900
-F 0 "#PWR029" H 2450 6650 60  0001 C CNN
-F 1 "GNDD" H 2450 6750 60  0000 C CNN
-F 2 "" H 2450 6900 60  0000 C CNN
-F 3 "" H 2450 6900 60  0000 C CNN
-	1    2450 6900
-	1    0    0    -1
-$EndComp
-$Comp
-L R R6
-U 1 1 557A2CF3
-P 2450 6050
-F 0 "R6" V 2530 6050 50  0000 C CNN
-F 1 "10k" V 2450 6050 50  0000 C CNN
-F 2 "Resistors_SMD:R_0603" V 2380 6050 30  0000 C CNN
-F 3 "" H 2450 6050 30  0000 C CNN
-F 4 "RMCF0603JT10K0" H 0   0   50  0001 C CNN "MPN"
-	1    2450 6050
-	1    0    0    1
-$EndComp
-$Comp
-L +9V #PWR030
-U 1 1 557A4EDD
-P 2450 5800
-F 0 "#PWR030" H 2450 5650 50  0001 C CNN
-F 1 "+9V" H 2450 5940 50  0000 C CNN
-F 2 "" H 2450 5800 60  0000 C CNN
-F 3 "" H 2450 5800 60  0000 C CNN
-	1    2450 5800
+P 2300 6400
+F 0 "#PWR029" H 2300 6150 60  0001 C CNN
+F 1 "GNDD" H 2300 6250 60  0000 C CNN
+F 2 "" H 2300 6400 60  0000 C CNN
+F 3 "" H 2300 6400 60  0000 C CNN
+	1    2300 6400
 	1    0    0    -1
 $EndComp
@@
 L Q_NMOS_GSD Q3
 U 1 1 557B0B85
-P 4200 6600
-F 0 "Q3" H 4100 6650 50  0000 R CNN
-F 1 "2N7002" V 4400 6750 50  0000 R CNN
-F 2 "Housings_SOT-23_SOT-143_TSOT-6:SOT-23" H 4400 6700 29  0000 C CNN
-F 3 "" H 4200 6600 60  0000 C CNN
-F 4 "2N7002P,215" H 0   0   50  0001 C CNN "MPN"
-	1    4200 6600
+P 4050 6100
+F 0 "Q3" H 3950 6150 50  0000 R CNN
+F 1 "2N7002" V 4250 6250 50  0000 R CNN
+F 2 "Housings_SOT-23_SOT-143_TSOT-6:SOT-23" H 4250 6200 29  0000 C CNN
+F 3 "" H 4050 6100 60  0000 C CNN
+F 4 "2N7002P,215" H -150 -500 50  0001 C CNN "MPN"
+	1    4050 6100
 	1    0    0    -1
 $EndComp
@@
 L GNDD #PWR031
 U 1 1 557B0B8B
-P 4300 6900
-F 0 "#PWR031" H 4300 6650 60  0001 C CNN
-F 1 "GNDD" H 4300 6750 60  0000 C CNN
-F 2 "" H 4300 6900 60  0000 C CNN
-F 3 "" H 4300 6900 60  0000 C CNN
-	1    4300 6900
-	1    0    0    -1
-$EndComp
-$Comp
-L R R7
-U 1 1 557B0B92
-P 4300 6050
-F 0 "R7" V 4380 6050 50  0000 C CNN
-F 1 "10k" V 4300 6050 50  0000 C CNN
-F 2 "Resistors_SMD:R_0603" V 4230 6050 30  0000 C CNN
-F 3 "" H 4300 6050 30  0000 C CNN
-F 4 "RMCF0603JT10K0" H 0   0   50  0001 C CNN "MPN"
-	1    4300 6050
-	1    0    0    1
-$EndComp
-$Comp
-L +9V #PWR032
-U 1 1 557B0B9A
-P 4300 5800
-F 0 "#PWR032" H 4300 5650 50  0001 C CNN
-F 1 "+9V" H 4300 5940 50  0000 C CNN
-F 2 "" H 4300 5800 60  0000 C CNN
-F 3 "" H 4300 5800 60  0000 C CNN
-	1    4300 5800
-	1    0    0    -1
-$EndComp
-$Comp
-L +9V #PWR033
-U 1 1 557B22CB
-P 2150 3300
-F 0 "#PWR033" H 2150 3150 50  0001 C CNN
-F 1 "+9V" H 2150 3440 50  0000 C CNN
-F 2 "" H 2150 3300 60  0000 C CNN
-F 3 "" H 2150 3300 60  0000 C CNN
-	1    2150 3300
-	1    0    0    -1
-$EndComp
-$Comp
-L +9V #PWR034
-U 1 1 557B2849
-P 2150 4000
-F 0 "#PWR034" H 2150 3850 50  0001 C CNN
-F 1 "+9V" H 2150 4140 50  0000 C CNN
-F 2 "" H 2150 4000 60  0000 C CNN
-F 3 "" H 2150 4000 60  0000 C CNN
-	1    2150 4000
-	1    0    0    -1
-$EndComp
-$Comp
-L +9V #PWR035
-U 1 1 557B3090
-P 2150 2200
-F 0 "#PWR035" H 2150 2050 50  0001 C CNN
-F 1 "+9V" H 2150 2340 50  0000 C CNN
-F 2 "" H 2150 2200 60  0000 C CNN
-F 3 "" H 2150 2200 60  0000 C CNN
-	1    2150 2200
-	1    0    0    -1
-$EndComp
-$Comp
-L +9V #PWR036
-U 1 1 557B39CA
-P 2150 1500
-F 0 "#PWR036" H 2150 1350 50  0001 C CNN
-F 1 "+9V" H 2150 1640 50  0000 C CNN
-F 2 "" H 2150 1500 60  0000 C CNN
-F 3 "" H 2150 1500 60  0000 C CNN
-	1    2150 1500
+P 4150 6400
+F 0 "#PWR031" H 4150 6150 60  0001 C CNN
+F 1 "GNDD" H 4150 6250 60  0000 C CNN
+F 2 "" H 4150 6400 60  0000 C CNN
+F 3 "" H 4150 6400 60  0000 C CNN
+	1    4150 6400
 	1    0    0    -1
 $EndComp
@@
 Text Notes 3000 5450 0    100  ~ 0
 STATUS LEDS
-Text GLabel 2650 6300 2    50   Output ~ 0
+Text GLabel 2500 5700 2    50   Output ~ 0
 RS485_RX_LED
 Text GLabel 8800 2800 2    50   Input ~ 0
 IO2
-Text GLabel 4500 6300 2    50   Output ~ 0
+Text GLabel 4350 5700 2    50   Output ~ 0
 RS485_TX_LED
 Text Notes 2950 1100 0    100  ~ 0
@@
 	2250 2300 2150 2300
 Wire Wire Line
-	2450 6800 2450 6900
-Wire Wire Line
-	2450 6200 2450 6400
-Wire Wire Line
-	2450 5900 2450 5800
-Wire Wire Line
-	2650 6300 2450 6300
-Wire Wire Line
-	2000 6600 2150 6600
-Wire Wire Line
-	4300 6800 4300 6900
-Wire Wire Line
-	4300 6200 4300 6400
-Wire Wire Line
-	4300 5900 4300 5800
-Wire Wire Line
-	4500 6300 4300 6300
-Wire Wire Line
-	3850 6600 4000 6600
+	2300 6300 2300 6400
+Wire Wire Line
+	2500 5700 2300 5700
+Wire Wire Line
+	1850 6100 2000 6100
+Wire Wire Line
+	4150 6300 4150 6400
+Wire Wire Line
+	4350 5700 4150 5700
+Wire Wire Line
+	3700 6100 3850 6100
 Wire Wire Line
 	2150 3400 2150 3300
@@
 Connection ~ 8150 1650
 Connection ~ 8650 2800
-Connection ~ 2450 6300
-Connection ~ 4300 6300
 $Comp
 L D D4
@@
 Wire Wire Line
 	9250 1700 9250 1600
-Text GLabel 2000 6600 0    50   BiDi ~ 0
+Text GLabel 1850 6100 0    50   BiDi ~ 0
 IO0/RXD
-Text GLabel 3850 6600 0    50   BiDi ~ 0
+Text GLabel 3700 6100 0    50   BiDi ~ 0
 IO1/TXD
+$Comp
+L +12V #PWR?
+U 1 1 560B0BA4
+P 4400 1750
+F 0 "#PWR?" H 4400 1600 50  0001 C CNN
+F 1 "+12V" H 4400 1890 50  0000 C CNN
+F 2 "" H 4400 1750 60  0000 C CNN
+F 3 "" H 4400 1750 60  0000 C CNN
+	1    4400 1750
+	1    0    0    -1
+$EndComp
+$Comp
+L +12V #PWR?
+U 1 1 560B1646
+P 2150 1500
+F 0 "#PWR?" H 2150 1350 50  0001 C CNN
+F 1 "+12V" H 2150 1640 50  0000 C CNN
+F 2 "" H 2150 1500 60  0000 C CNN
+F 3 "" H 2150 1500 60  0000 C CNN
+	1    2150 1500
+	1    0    0    -1
+$EndComp
+$Comp
+L +12V #PWR?
+U 1 1 560B1B05
+P 2150 2200
+F 0 "#PWR?" H 2150 2050 50  0001 C CNN
+F 1 "+12V" H 2150 2340 50  0000 C CNN
+F 2 "" H 2150 2200 60  0000 C CNN
+F 3 "" H 2150 2200 60  0000 C CNN
+	1    2150 2200
+	1    0    0    -1
+$EndComp
+$Comp
+L +12V #PWR?
+U 1 1 560B1E7A
+P 2150 3300
+F 0 "#PWR?" H 2150 3150 50  0001 C CNN
+F 1 "+12V" H 2150 3440 50  0000 C CNN
+F 2 "" H 2150 3300 60  0000 C CNN
+F 3 "" H 2150 3300 60  0000 C CNN
+	1    2150 3300
+	1    0    0    -1
+$EndComp
+$Comp
+L +12V #PWR?
+U 1 1 560B204D
+P 2150 4000
+F 0 "#PWR?" H 2150 3850 50  0001 C CNN
+F 1 "+12V" H 2150 4140 50  0000 C CNN
+F 2 "" H 2150 4000 60  0000 C CNN
+F 3 "" H 2150 4000 60  0000 C CNN
+	1    2150 4000
+	1    0    0    -1
+$EndComp
+Wire Wire Line
+	2300 5700 2300 5900
+Wire Wire Line
+	4150 5700 4150 5900
+$Comp
+L +12V #PWR?
+U 1 1 560B7499
+P 4400 3550
+F 0 "#PWR?" H 4400 3400 50  0001 C CNN
+F 1 "+12V" H 4400 3690 50  0000 C CNN
+F 2 "" H 4400 3550 60  0000 C CNN
+F 3 "" H 4400 3550 60  0000 C CNN
+	1    4400 3550
+	1    0    0    -1
+$EndComp
+$Comp
+L +12V #PWR?
+U 1 1 560B74CD
+P 4950 3550
+F 0 "#PWR?" H 4950 3400 50  0001 C CNN
+F 1 "+12V" H 4950 3690 50  0000 C CNN
+F 2 "" H 4950 3550 60  0000 C CNN
+F 3 "" H 4950 3550 60  0000 C CNN
+	1    4950 3550
+	1    0    0    -1
+$EndComp
 $EndSCHEMATC

Commit message: sch: fixing MOSFET + new BOM exported
Parts:
- C3: value 100nF X7R -> 100nF
- Q2, Q3: value 2N7002 -> BSS84; symbol Q_NMOS_GSD -> Q_PMOS_GSD; MPN 2N7002P,215 -> BSS84
- R10, R8: value 10k -> 10K
- R2, R3, R4, R5: value 1K -> 330R
Connections:
- net +12V: no longer R2.2, R3.2, R4.2, R5.2
- net +3V3: now also Q2.2 (S), Q3.2 (S)
- net GNDD: now also J1.11, J1.9, J2.11, J2.9; no longer Q2.2 (S), Q3.2 (S)
- net RS485_RX_LED: now also R2.2, R4.2; no longer J1.11, J2.11
- net RS485_TX_LED: now also R3.2, R5.2; no longer J1.9, J2.9

Commit message: fixing user led voltage
Parts:
- R2, R3, R4, R5: MPN ESR03EZPJ102 -> RMCF0603JT330R
Changed lines of the file:
@@
 F 2 "Resistors_SMD:R_0603" V 2330 3400 30  0001 C CNN
 F 3 "" H 2400 3400 30  0000 C CNN
-F 4 "ESR03EZPJ102" H 0   0   50  0001 C CNN "MPN"
+F 4 "RMCF0603JT330R" H 0   0   50  0001 C CNN "MPN"
 	1    2400 3400
 	0    1    -1   0
@@
 F 2 "Resistors_SMD:R_0603" V 2330 1600 30  0001 C CNN
 F 3 "" H 2400 1600 30  0000 C CNN
-F 4 "ESR03EZPJ102" H 0   0   50  0001 C CNN "MPN"
+F 4 "RMCF0603JT330R" H 0   0   50  0001 C CNN "MPN"
 	1    2400 1600
 	0    1    -1   0
@@
 F 2 "Resistors_SMD:R_0603" V 2330 4100 30  0001 C CNN
 F 3 "" H 2400 4100 30  0000 C CNN
-F 4 "ESR03EZPJ102" H 0   0   50  0001 C CNN "MPN"
+F 4 "RMCF0603JT330R" H 0   0   50  0001 C CNN "MPN"
 	1    2400 4100
 	0    1    -1   0
@@
 F 2 "Resistors_SMD:R_0603" V 2330 2300 30  0001 C CNN
 F 3 "" H 2400 2300 30  0000 C CNN
-F 4 "ESR03EZPJ102" H 0   0   50  0001 C CNN "MPN"
+F 4 "RMCF0603JT330R" H 0   0   50  0001 C CNN "MPN"
 	1    2400 2300
 	0    1    -1   0
