File: hw-design/board/arduino-connectors.sch (KiCad schematic (older format))
At the start: 15 parts, among them P1 Power, P2 Analog, P3 Digital, P4 Digital, P5 Hole, P6 Hole, P7 Hole, P8 Hole, Q1 2N7002

Commit message: add header MPN to BOM
Parts:
- P1, P4: MPN (none) -> PREC008SFAN-RC
- P2: MPN (none) -> PREC006SFAN-RC
- P3: MPN (none) -> PREC010SFAN-RC
Changed lines of the file:
@@
 F 2 "Socket_Arduino_Uno:Socket_Strip_Arduino_1x08" V 5450 2000 60  0001 C CNN
 F 3 "" H 5450 2000 60  0000 C CNN
+F 4 "PREC008SFAN-RC" H 5450 2000 60  0001 C CNN "MPN"
 	1    5450 2000
 	-1   0    0    -1
@@
 F 2 "Socket_Arduino_Uno:Socket_Strip_Arduino_1x06" V 5450 2950 60  0001 C CNN
 F 3 "" H 5450 2950 60  0000 C CNN
+F 4 "PREC006SFAN-RC" H 5450 2950 60  0001 C CNN "MPN"
 	1    5450 2950
 	-1   0    0    -1
@@
 F 2 "Socket_Arduino_Uno:Socket_Strip_Arduino_1x10" V 7200 1950 60  0001 C CNN
 F 3 "" H 7200 1950 60  0000 C CNN
+F 4 "PREC010SFAN-RC" H 7200 1950 60  0001 C CNN "MPN"
 	1    7200 1950
 	1    0    0    -1
@@
 F 2 "Socket_Arduino_Uno:Socket_Strip_Arduino_1x08" V 7200 3000 60  0001 C CNN
 F 3 "" H 7200 3000 60  0000 C CNN
+F 4 "PREC008SFAN-RC" H 7200 3000 60  0001 C CNN "MPN"
 	1    7200 3000
 	1    0    0    -1
